Commit message: Update rover.urdf.xacro

File: scort/urdf/rover.urdf.xacro (robot description, xacro)
@@ -2,17 +2,19 @@
 <robot xmlns:xacro="http://www.ros.org/wiki/xacro" name="rover">
 <link name="base_footprint"/>
-<link name="base">
+<link name="base_link">
     <inertial>
         <origin xyz="0.0 0.0 0.0" rpy="0.0 0.0 0.0"/>
         <mass value="1.0"/>
-        <inertia ixx="0.4" ixy="0.0" ixz="0.0" iyy="0.4" iyz="0.0" izz="0.2"/>
-    </inertial>
+        <inertia ixx="0.4" ixy="0.0" ixz="0.0"
+                 iyy="0.4" iyz="0.0"
+                 izz="0.2"/>
+    </inertial>a
     <visual name="">
         <origin xyz="0.0 0.0 0.0" rpy="0.0 0.0 0.0"/>
         <geometry>
-            <box size="0.7 0.7 0.1"/>
+            <box size="0.8 0.7 0.1"/>
         </geometry>
         <material name="">
-            <color rgba="0.0 0.6 1.0 1.0"/>
+            <color rgba="1.0 0.0 0.0 1.0"/>
             <texture filename=""/>
         </material>
@@ -26,15 +28,15 @@
 </link>
 <joint name="base_joint" type="fixed">
-        <origin xyz="0.0 0.0 0.135" rpy="0.0 0.0 0.0"/>
-        <parent link="base_footprint"/>
-        <child link="base"/>
-        <axis xyz="0.0 0.0 0.0"/>
+    <origin xyz="0.0 0.0 0.135" rpy="0.0 0.0 0.0"/>
+    <parent link="base_footprint"/>
+    <child link="base_link"/>
+    <axis xyz="0.0 0.0 0.0"/>
 </joint>
-    <!--Wheels-->
-<xacro:macro name="tyre" params="name x y p">
-    <link name="Wheel_$(name)_link">
+<!-- All Wheel links and joints -->
+<xacro:macro name="wheel" params="name x y">
+    <link name="wheel_${name}_link">
         <inertial>
             <origin xyz="0.0 0.0 0.0" rpy="0.0 0.0 0.0"/>
-            <mass value="0.0"/>
+            <mass value="0.5"/>
             <inertia ixx="0.0" ixy="0.0" ixz="0.0" iyy="0.0" iyz="0.0" izz="0.0"/>
         </inertial>
@@ -42,9 +44,8 @@
             <origin xyz="0.0 0.0 0.0" rpy="0.0 0.0 0.0"/>
             <geometry>
-                <cylinder radius="0.1" length="0.1"/>
+                <mesh filename="package://mobile_robot/meshes/left_tire.stl" scale="0.005 0.005 0.005"/>
             </geometry>
-            <material name="">
-                <color rgba="0.25 0.5 0.7 1.0"/>
-                <texture filename=""/>
+            <material name="black">
+                <color rgba=".0 .0 0.0 1.0"/>
             </material>
         </visual>
@@ -52,19 +53,19 @@
             <origin xyz="0.0 0.0 0.0" rpy="0.0 0.0 0.0"/>
             <geometry>
-                <cylinder radius="0.0" length="0.0"/>
+                <mesh filename="package://mobile_robot/meshes/left_tire.stl" scale="0.005 0.005 0.005"/>
             </geometry>
         </collision>
     </link>
-    <joint name="$(name)_wheel_joint" type="continuous">
-        <origin xyz="${x} ${y} 0.0" rpy="1.57 1.5708 ${p}"/>
-        <parent link="base"/>
-        <child link="Wheel_$(name)_link"/>
-        <axis xyz="0.0 0.0 1.0"/>
-        <limit lower="0.0" upper="0.0" effort="0.0" velocity="0.0"/>
+    <joint name="wheel_${name}_joint" type="continuous">
+        <origin xyz="${x} ${y} .0" rpy="0 0.0 0.0"/>
+        <parent link="base_link"/>
+        <child link="wheel_${name}_link"/>
+        <axis xyz=".0 .0 1.0"/>
     </joint>
 </xacro:macro>
-<xacro:tyre name = "rear_left" x="0.3" y="-0.40" p="0.785398"/>
-<xacro:tyre name = "front_left" x="-0.3" y="-0.40" p=" -0.785398"/>
-<xacro:tyre name = "front_right" x="-0.3" y="-0.40" p=" -0.785398"/>
-<xacro:tyre name = "rear_right" x="0.3" y="0.40" p=" 0.785398"/>
+<!-- Wheel Creating using macros -->
+<xacro:wheel name="rear_right"  x="0.250" y =" 0.40"/>
+<xacro:wheel name="front_right" x="-0.250" y =" 0.40"/>
+<xacro:wheel name="front_left"  x="-0.250" y =" -0.40"/>
+<xacro:wheel name="rear_left"   x="0.250" y =" -0.40"/>
 </robot>

Commit message: Update rover.urdf.xacro

File: scort/urdf/rover.urdf.xacro (robot description, xacro)
@@ -2,19 +2,17 @@
 <robot xmlns:xacro="http://www.ros.org/wiki/xacro" name="rover">
 <link name="base_footprint"/>
-<link name="base_link">
+<link name="base">
     <inertial>
         <origin xyz="0.0 0.0 0.0" rpy="0.0 0.0 0.0"/>
         <mass value="1.0"/>
-        <inertia ixx="0.4" ixy="0.0" ixz="0.0"
-                 iyy="0.4" iyz="0.0"
-                 izz="0.2"/>
-    </inertial>a
+        <inertia ixx="0.4" ixy="0.0" ixz="0.0" iyy="0.4" iyz="0.0" izz="0.2"/>
+    </inertial>
     <visual name="">
         <origin xyz="0.0 0.0 0.0" rpy="0.0 0.0 0.0"/>
         <geometry>
-            <box size="0.8 0.7 0.1"/>
+            <box size="0.7 0.7 0.1"/>
         </geometry>
         <material name="">
-            <color rgba="1.0 0.0 0.0 1.0"/>
+            <color rgba="0.0 0.6 1.0 1.0"/>
             <texture filename=""/>
         </material>
@@ -28,15 +26,15 @@
 </link>
 <joint name="base_joint" type="fixed">
-    <origin xyz="0.0 0.0 0.135" rpy="0.0 0.0 0.0"/>
-    <parent link="base_footprint"/>
-    <child link="base_link"/>
-    <axis xyz="0.0 0.0 0.0"/>
+        <origin xyz="0.0 0.0 0.135" rpy="0.0 0.0 0.0"/>
+        <parent link="base_footprint"/>
+        <child link="base"/>
+        <axis xyz="0.0 0.0 0.0"/>
 </joint>
-<!-- All Wheel links and joints -->
-<xacro:macro name="wheel" params="name x y">
-    <link name="wheel_${name}_link">
+    <!--Wheels-->
+<xacro:macro name="tyre" params="name x y p">
+    <link name="Wheel_$(name)_link">
         <inertial>
             <origin xyz="0.0 0.0 0.0" rpy="0.0 0.0 0.0"/>
-            <mass value="0.5"/>
+            <mass value="0.0"/>
             <inertia ixx="0.0" ixy="0.0" ixz="0.0" iyy="0.0" iyz="0.0" izz="0.0"/>
         </inertial>
@@ -44,8 +42,9 @@
             <origin xyz="0.0 0.0 0.0" rpy="0.0 0.0 0.0"/>
             <geometry>
-                <mesh filename="package://mobile_robot/meshes/left_tire.stl" scale="0.005 0.005 0.005"/>
+                <cylinder radius="0.1" length="0.1"/>
             </geometry>
-            <material name="black">
-                <color rgba=".0 .0 0.0 1.0"/>
+            <material name="">
+                <color rgba="0.25 0.5 0.7 1.0"/>
+                <texture filename=""/>
             </material>
         </visual>
@@ -53,19 +52,19 @@
             <origin xyz="0.0 0.0 0.0" rpy="0.0 0.0 0.0"/>
             <geometry>
-                <mesh filename="package://mobile_robot/meshes/left_tire.stl" scale="0.005 0.005 0.005"/>
+                <cylinder radius="0.0" length="0.0"/>
             </geometry>
         </collision>
     </link>
-    <joint name="wheel_${name}_joint" type="continuous">
-        <origin xyz="${x} ${y} .0" rpy="0 0.0 0.0"/>
-        <parent link="base_link"/>
-        <child link="wheel_${name}_link"/>
-        <axis xyz=".0 .0 1.0"/>
+    <joint name="$(name)_wheel_joint" type="continuous">
+        <origin xyz="${x} ${y} 0.0" rpy="1.57 1.5708 ${p}"/>
+        <parent link="base"/>
+        <child link="Wheel_$(name)_link"/>
+        <axis xyz="0.0 0.0 1.0"/>
+        <limit lower="0.0" upper="0.0" effort="0.0" velocity="0.0"/>
     </joint>
 </xacro:macro>
-<!-- Wheel Creating using macros -->
-<xacro:wheel name="rear_right"  x="0.250" y =" 0.40"/>
-<xacro:wheel name="front_right" x="-0.250" y =" 0.40"/>
-<xacro:wheel name="front_left"  x="-0.250" y =" -0.40"/>
-<xacro:wheel name="rear_left"   x="0.250" y =" -0.40"/>
+<xacro:tyre name = "rear_left" x="0.3" y="-0.40" p="0.785398"/>
+<xacro:tyre name = "front_left" x="-0.3" y="-0.40" p=" -0.785398"/>
+<xacro:tyre name = "front_right" x="-0.3" y="-0.40" p=" -0.785398"/>
+<xacro:tyre name = "rear_right" x="0.3" y="0.40" p=" 0.785398"/>
 </robot>
